File: PCB V2/Kicad/OOK48_PICO.kicad_pcb (KiCad board)
At the start: 2 copper layers, 98.7 x 56.4 mm, 28 parts, among them J1 Conn_01x14_Socket, J2 Conn_01x04_Socket, J3 Conn_01x04_Pin, J4 Conn_01x05_Pin, J5 Conn_01x02_Pin, J6 Conn_01x02_Pin, Q1 DMN3404L, Q2 DMN3404L, U1 LTC4054ES5-4.2

Commit message: Update PCB
Parts:
- removed R6, R7: 100K, Capacitor_SMD:C_0805_2012Metric_Pad1.18x1.45mm_HandSolder
- R1: value 10K -> 1K5
- moved H3 2.00 mm to (188.5, 118.5)
- moved H4 2.00 mm to (188.5, 69.0)
- moved J1 2.00 mm to (189.4, 110.2)
Connections:
- A1 pad 32: /GP27-BAT -> unconnected-(A1-GPIO27_ADC1-Pad32)
Routing:
- net /GP27-BAT: track 36.0 -> 0.00 mm, vias 1 -> 0
- net unconnected-(A1-GPIO27_ADC1-Pad32): track 0.00 -> 15.3 mm, vias 0 -> 1
- net /IO8-D/C: track 79.1 -> 76.9 mm
- net VSYS: track 108.8 -> 106.8 mm
- net GND: track 284.6 -> 282.6 mm
- net /IO9-CS: track 81.5 -> 79.5 mm
- net /IO16-TCS: track 58.1 -> 56.1 mm
- net /IO12-MISO: track 110.0 -> 108.0 mm
- net /IO17-TIRQ: track 68.4 -> 66.4 mm
- net /IO18-LED: track 58.1 -> 56.2 mm
- net /IO15-RST: track 58.4 -> 56.5 mm
Other:
- board size 98.7 x 56.4 mm -> 96.8 x 56.4 mm
