File: PCB V2/Kicad/OOK48_PICO.kicad_sch (KiCad schematic)
At the start: 28 parts, among them J1 Conn_01x14_Socket, J2 Conn_01x04_Socket, J3 Conn_01x04_Pin, J4 Conn_01x05_Pin, J5 Conn_01x02_Pin, J6 Conn_01x02_Pin, Q1 DMN3404L, Q2 DMN3404L, U1 LTC4054ES5-4.2

Commit message: Update PCB
Parts:
- removed R6, R7: 100K, Capacitor_SMD:C_0805_2012Metric_Pad1.18x1.45mm_HandSolder, symbol Device:R
Connections:
- net GP27-BAT: no longer names the net of A1.32 (GPIO27_ADC1)
- no-connect marks 13 -> 14
Changed lines of the file:
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@@
-	)
-	(junction
-		(at 102.87 52.07)
-		(diameter 0)
-		(color 0 0 0 0)
 	)
 	(junction
@@
 	)
 	(junction
-		(at 97.79 62.23)
-		(diameter 0)
-		(color 0 0 0 0)
-	)
-	(junction
 		(at 54.61 27.94)
 		(diameter 0)
@@
 	)
 	(junction
-		(at 102.87 44.45)
-		(diameter 0)
-		(color 0 0 0 0)
-	)
-	(junction
 		(at 90.17 62.23)
 		(diameter 0)
@@
 	)
 	(no_connect
+		(at 162.56 110.49)
+	)
+	(no_connect
 		(at 116.84 113.03)
 	)
@@
 	(wire
 		(pts
-			(xy 102.87 44.45) (xy 107.95 44.45)
-		)
-		(stroke
-			(width 0)
-			(type default)
-		)
-	)
-	(wire
-		(pts
 			(xy 107.95 105.41) (xy 116.84 105.41)
 		)
@@
 	(wire
 		(pts
-			(xy 95.25 44.45) (xy 102.87 44.45)
-		)
-		(stroke
-			(width 0)
-			(type default)
-		)
-	)
-	(wire
-		(pts
-			(xy 97.79 62.23) (xy 102.87 62.23)
+			(xy 95.25 44.45) (xy 107.95 44.45)
 		)
 		(stroke
@@
 	(wire
 		(pts
-			(xy 162.56 110.49) (xy 166.37 110.49)
-		)
-		(stroke
-			(width 0)
-			(type default)
-		)
-	)
-	(wire
-		(pts
 			(xy 60.96 62.23) (xy 76.2 62.23)
 		)
@@
 	(wire
 		(pts
-			(xy 113.03 52.07) (xy 102.87 52.07)
-		)
-		(stroke
-			(width 0)
-			(type default)
-		)
-	)
-	(wire
-		(pts
 			(xy 41.91 181.61) (xy 41.91 152.4)
 		)
@@
 	(wire
 		(pts
-			(xy 102.87 52.07) (xy 102.87 53.34)
-		)
-		(stroke
-			(width 0)
-			(type default)
-		)
-	)
-	(wire
-		(pts
 			(xy 231.14 88.9) (xy 236.22 88.9)
 		)
@@
 		(pts
 			(xy 83.82 181.61) (xy 90.17 181.61)
-		)
-		(stroke
-			(width 0)
-			(type default)
-		)
-	)
-	(wire
-		(pts
-			(xy 102.87 60.96) (xy 102.87 62.23)
 		)
 		(stroke
@@
 			)
 			(justify right)
-		)
-	)
-	(label "GP27-BAT"
-		(at 166.37 110.49 0)
-		(effects
-			(font
-				(size 1.27 1.27)
-			)
-			(justify left)
 		)
 	)
@@
 			)
 			(justify right)
-		)
-	)
-	(label "GP27-BAT"
-		(at 113.03 52.07 0)
-		(effects
-			(font
-				(size 1.27 1.27)
-			)
-			(justify left)
 		)
 	)
@@
 	)
 	(symbol
-		(lib_id "Device:R")
-		(at 102.87 57.15 0)
-		(unit 1)
-		(exclude_from_sim no)
-		(in_bom yes)
-		(on_board yes)
-		(dnp no)
-		(property "Reference" "R7"
-			(at 104.648 55.88 0)
-			(effects
-				(font
-					(size 1.27 1.27)
-				)
-				(justify left)
-			)
-		)
-		(property "Value" "100K"
-			(at 104.648 58.928 0)
-			(effects
-				(font
-					(size 1.27 1.27)
-				)
-				(justify left)
-			)
-		)
-		(property "Footprint" "Capacitor_SMD:C_0805_2012Metric_Pad1.18x1.45mm_HandSolder"
-			(at 101.092 57.15 90)
-			(effects
-				(font
-					(size 1.27 1.27)
-				)
-				(hide yes)
-			)
-		)
-		(property "Datasheet" "~"
-			(at 102.87 57.15 0)
-			(effects
-				(font
-					(size 1.27 1.27)
-				)
-				(hide yes)
-			)
-		)
-		(property "Description" "Resistor"
-			(at 102.87 57.15 0)
-			(effects
-				(font
-					(size 1.27 1.27)
-				)
-				(hide yes)
-			)
-		)
-		(pin "2"
-		)
-		(pin "1"
-		)
-		(instances
-			(project "OOK48_PICO"
-				(path "/9e450d93-50b3-4aad-bb89-e951560c22c5"
-					(reference "R7")
-					(unit 1)
-				)
-			)
-		)
-	)
-	(symbol
 		(lib_id "power:+5V")
 		(at 139.7 49.53 0)
@@
 					(unit 1)
 				)
-			)
-		)
-	)
-	(symbol
-		(lib_id "Device:R")
-		(at 102.87 48.26 0)
-		(unit 1)
-		(exclude_from_sim no)
-		(in_bom yes)
-		(on_board yes)
-		(dnp no)
-		(property "Reference" "R6"
-			(at 104.648 46.99 0)
-			(effects
-				(font
-					(size 1.27 1.27)
-				)
-				(justify left)
-			)
-		)
-		(property "Value" "100K"
-			(at 104.648 49.784 0)
-			(effects
-				(font
-					(size 1.27 1.27)
-				)
-				(justify left)
-			)
-		)
-		(property "Footprint" "Capacitor_SMD:C_0805_2012Metric_Pad1.18x1.45mm_HandSolder"
-			(at 101.092 48.26 90)
-			(effects
-				(font
-					(size 1.27 1.27)
-				)
-				(hide yes)
-			)
-		)
-		(property "Datasheet" "~"
-			(at 102.87 48.26 0)
-			(effects
-				(font
-					(size 1.27 1.27)
-				)
-				(hide yes)
-			)
-		)
-		(property "Description" "Resistor"
-			(at 102.87 48.26 0)
-			(effects
-				(font
-					(size 1.27 1.27)
-				)
-				(hide yes)
-			)
-		)
-		(pin "2"
-		)
-		(pin "1"
-		)
-		(instances
-			(project "OOK48_PICO"
-				(path "/9e450d93-50b3-4aad-bb89-e951560c22c5"
-					(reference "R6")
-					(unit 1)
-				)
